File: KiCad/Super_Mini_Mega Tester.kicad_pcb (KiCad board)
At the start: 2 copper layers, 99.9 x 99.7 mm, 45 parts, among them J1 Conn_01x05, J2 Conn_02x20_Odd_Even, J3 Conn_02x20_Odd_Even, J4 Conn_01x04, J5 Conn_01x05, Q1 2N7000, Q2 2N7000, SW1 RotaryEncoder_Switch, U1 ESP32-C3-Super-Mini, U2 MCP23017_SP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

Commit message: Add files via upload
Other:
- board text added: "+5V"
- board text added: "1 40"
- board text added: "20 21"
- board text removed: "1 2"
- board text removed: "39 40"
Changed lines of the file:
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@@
+		)
+	)
+	(gr_text "GND"
+		(at 106.7008 121.6748 90)
+		(layer "F.SilkS")
+		(effects
+			(font
+				(size 1 1)
+				(thickness 0.15)
+			)
+			(justify left bottom)
 		)
 	)
@@
 		)
 	)
+	(gr_text "+5V"
+		(at 37.4308 100.1984 0)
+		(layer "F.SilkS")
+		(effects
+			(font
+				(size 1 1)
+				(thickness 0.15)
+			)
+			(justify left bottom)
+		)
+	)
 	(gr_text "Menu"
 		(at 122.724 49.373 0)
@@
 		)
 	)
+	(gr_text "+5V"
+		(at 120.3872 116.9624 0)
+		(layer "F.SilkS")
+		(effects
+			(font
+				(size 1 1)
+				(thickness 0.15)
+			)
+			(justify left bottom)
+		)
+	)
 	(gr_text "9"
 		(at 54.326 56.346 90)
@@
 		)
 	)
-	(gr_text "1\n\n2"
-		(at 118.653 59.074 90)
+	(gr_text "GND"
+		(at 37.5832 97.7092 0)
+		(layer "F.SilkS")
+		(effects
+			(font
+				(size 1 1)
+				(thickness 0.15)
+			)
+			(justify left bottom)
+		)
+	)
+	(gr_text "+5V"
+		(at 60.1892 100.554 0)
+		(layer "F.SilkS")
+		(effects
+			(font
+				(size 1 1)
+				(thickness 0.15)
+			)
+			(justify left bottom)
+		)
+	)
+	(gr_text "1\n\n40"
+		(at 118.653 58.82 90)
 		(layer "F.SilkS")
 		(effects
@@
 		)
 	)
-	(gr_text "1\n\n2"
-		(at 58.201 59.201 90)
-		(layer "F.SilkS")
-		(effects
-			(font
-				(size 1 1)
-				(thickness 0.15)
-			)
-			(justify left bottom)
-		)
-	)
-	(gr_text "39\n\n40\n"
-		(at 118.816 112.502 90)
+	(gr_text "1\n\n40"
+		(at 58.3026 58.947 90)
+		(layer "F.SilkS")
+		(effects
+			(font
+				(size 1 1)
+				(thickness 0.15)
+			)
+			(justify left bottom)
+		)
+	)
+	(gr_text "GND"
+		(at 120.438 114.4224 0)
+		(layer "F.SilkS")
+		(effects
+			(font
+				(size 1 1)
+				(thickness 0.15)
+			)
+			(justify left bottom)
+		)
+	)
+	(gr_text "20\n\n21\n"
+		(at 118.6636 112.6036 90)
 		(layer "F.SilkS")
 		(effects
@@
 		)
 	)
+	(gr_text "+5V"
+		(at 109.3424 121.8272 90)
+		(layer "F.SilkS")
+		(effects
+			(font
+				(size 1 1)
+				(thickness 0.15)
+			)
+			(justify left bottom)
+		)
+	)
 	(gr_text "Output"
 		(at 62.449 74.69 90)
@@
 		)
 	)
+	(gr_text "GND"
+		(at 60.9004 96.998 0)
+		(layer "F.SilkS")
+		(effects
+			(font
+				(size 1 1)
+				(thickness 0.15)
+			)
+			(justify left bottom)
+		)
+	)
 	(gr_text "5V"
 		(at 101.796 34.054 90)
@@
 		)
 	)
-	(gr_text "39\n\n40\n"
-		(at 58.491 112.629 90)
+	(gr_text "20\n\n21"
+		(at 58.2878 112.9338 90)
 		(layer "F.SilkS")
 		(effects
@@
 		)
 	)
+	(gr_text "GND"
+		(at 98.086 98.2172 0)
+		(layer "F.SilkS")
+		(effects
+			(font
+				(size 1 1)
+				(thickness 0.15)
+			)
+			(justify left bottom)
+		)
+	)
 	(gr_text "4"
 		(at 53.183 31.327 90)
@@
 				(thickness 0.15)
 			)
+			(justify left bottom)
+		)
+	)
+	(gr_text "+5V"
+		(at 97.832 100.9604 0)
+		(layer "F.SilkS")
+		(effects
+			(font
+				(size 1 1)
+				(thickness 0.15)
+			)
