File: KiCad/Super_Mini_Mega Tester.kicad_sch (KiCad schematic)
At the start: 45 parts, among them J1 Conn_01x05, J2 Conn_02x20_Odd_Even, J3 Conn_02x20_Odd_Even, J4 Conn_01x04, J5 Conn_01x05, Q1 2N7000, Q2 2N7000, SW1 RotaryEncoder_Switch, U1 ESP32-C3-Super-Mini, U2 MCP23017_SP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

Commit message: Add files via upload
Other:
- note added: "Note: 40 pin header pin numbers are assigned as shown, ignoring actual footprint pin numbers."
- note added: "Pin 1"
- note added: "Pin 20"
- note added: "Pin 21"
- note added: "Pin 40"
Changed lines of the file:
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@@
+		)
+	)
+	(text "Pin 20"
+		(exclude_from_sim no)
+		(at 250.444 88.9 0)
+		(effects
+			(font
+				(size 1.27 1.27)
+			)
+			(justify left bottom)
 		)
 	)
@@
 		)
 	)
+	(text "Pin 21"
+		(exclude_from_sim no)
+		(at 316.484 88.9 0)
+		(effects
+			(font
+				(size 1.27 1.27)
+			)
+			(justify left bottom)
+		)
+	)
 	(text "A2"
 		(exclude_from_sim no)
@@
 		)
 	)
+	(text "Pin 21"
+		(exclude_from_sim no)
+		(at 264.668 88.9 0)
+		(effects
+			(font
+				(size 1.27 1.27)
+			)
+			(justify left bottom)
+		)
+	)
 	(text "GPIO10"
 		(exclude_from_sim no)
@@
 		)
 	)
+	(text "Pin 40"
+		(exclude_from_sim no)
+		(at 264.414 40.64 0)
+		(effects
+			(font
+				(size 1.27 1.27)
+			)
+			(justify left bottom)
+		)
+	)
+	(text "Pin 40"
+		(exclude_from_sim no)
+		(at 316.23 40.64 0)
+		(effects
+			(font
+				(size 1.27 1.27)
+			)
+			(justify left bottom)
+		)
+	)
+	(text "Note: 40 pin header pin numbers are assigned as shown, ignoring actual footprint pin numbers."
+		(exclude_from_sim no)
+		(at 240.538 94.996 0)
+		(effects
+			(font
+				(size 1.27 1.27)
+			)
+			(justify left bottom)
+		)
+	)
 	(text "A2"
 		(exclude_from_sim no)
@@
 		)
 	)
+	(text "Pin 20"
+		(exclude_from_sim no)
+		(at 302.006 88.9 0)
+		(effects
+			(font
+				(size 1.27 1.27)
+			)
+			(justify left bottom)
+		)
+	)
 	(text "Inputs"
 		(exclude_from_sim no)
@@
 		)
 	)
+	(text "Pin 1"
+		(exclude_from_sim no)
+		(at 303.53 40.64 0)
+		(effects
+			(font
+				(size 1.27 1.27)
+			)
+			(justify left bottom)
+		)
+	)
 	(text "GPIO2"
 		(exclude_from_sim no)
@@
 			(font
 				(size 2.54 2.54)
+			)
+			(justify left bottom)
+		)
+	)
+	(text "Pin 1"
+		(exclude_from_sim no)
+		(at 251.714 40.64 0)
+		(effects
+			(font
+				(size 1.27 1.27)
 			)
 			(justify left bottom)
@@
 	)
 	(symbol
+		(lib_name "Conn_02x20_Odd_Even_1")
 		(lib_id "Connector_Generic:Conn_02x20_Odd_Even")
 		(at 259.08 63.5 0)
